Commit message: fix urdf and IK dummy ujang

File: milestone3/arm/urdf/dump_kaki_ujang.urdf (robot description, URDF)
Before this commit: robot dump_kaki_ujang, 5 links, 4 joints
Links:
- link coxa_link: geometry visual cylinder length=0.25 radius=0.1
Joints:
- joint joint_end_effector: origin xyz=0.1 0 -0.6149 rpy=0 0 0 -> xyz=0 0 -0.7149 rpy=0 0 0
- joint joint_fermur: axis 0 1 0 -> 0 -1 0; origin xyz=0.25 0 -0.1 rpy=0 0 0 -> xyz=0.25 0 0 rpy=0 0 0
- joint joint_tibia: axis 0 1 0 -> 0 -1 0
